File: ultra96v2_glasses.kicad_pcb (KiCad board)
At the start: 2 copper layers, 85 x 54 mm, 12 parts, among them J1 61083-063402LF, J1 PMOD_M_2X6, J2 10075024-G01-20ULF, J3 1-1734248-5, J4 1-1734248-5

Commit message: update
Parts:
- removed the J1 at (131.5, 112.8)
- removed the J1 at (110.0, 112.8)
- removed the REF** at (171.8, 146.0)
- removed the REF** at (113.0, 146.0)
- added C1: 10uF, Capacitor_SMD:C_0603_1608Metric, F.Cu at (148.5, 191.0)
- added C10: 0.1uF, Capacitor_SMD:C_0603_1608Metric, F.Cu at (144.3, 188.5)
- added C11: 0.1uF, Capacitor_SMD:C_0603_1608Metric, F.Cu at (140.5, 193.1)
- added C12: 0.1uF, Capacitor_SMD:C_0603_1608Metric, F.Cu at (148.4, 186.0)
- added C13: 2.2uF, Capacitor_SMD:C_0603_1608Metric, F.Cu at (161.2, 178.0)
- added C14: 220pF/25V, Capacitor_SMD:C_0603_1608Metric, F.Cu at (156.5, 191.0)
- added C15: 4.7uF 25V, Capacitor_SMD:C_0603_1608Metric, F.Cu at (169.2, 183.5)
- added C16: 0.1uF, Capacitor_SMD:C_0603_1608Metric, F.Cu at (180.6, 172.5)
- added C17: 0.1uF, Capacitor_SMD:C_0603_1608Metric, F.Cu at (160.5, 190.6)
- added C18: 0.1uF, Capacitor_SMD:C_0603_1608Metric, F.Cu at (164.4, 188.1)
- added C19: 0.1uF, Capacitor_SMD:C_0603_1608Metric, F.Cu at (136.5, 195.7)
- added C2: 10uF, Capacitor_SMD:C_0603_1608Metric, F.Cu at (133.9, 190.6)
- added C20: 0.1uF, Capacitor_SMD:C_0603_1608Metric, F.Cu at (148.5, 193.5)
- added C21: 0.1uF, Capacitor_SMD:C_0603_1608Metric, F.Cu at (175.5, 167.5)
- added C22: 10uF 25V, Capacitor_SMD:C_0603_1608Metric, F.Cu at (165.2, 178.0)
- added C23: 10uF 25V, Capacitor_SMD:C_0603_1608Metric, F.Cu at (181.3, 159.1)
- added C24: 4.7uF, Capacitor_SMD:C_0603_1608Metric, F.Cu at (161.2, 180.5)
- added C25: 4.7uF, Capacitor_SMD:C_0603_1608Metric, F.Cu at (175.5, 165.0)
- added C26: 0.1uF, Capacitor_SMD:C_0603_1608Metric, F.Cu at (144.5, 196.0)
- added C27: 0.1uF, Capacitor_SMD:C_0603_1608Metric, F.Cu at (152.4, 188.5)
- added C28: 0.1uF 25V, Capacitor_SMD:C_0603_1608Metric, F.Cu at (128.4, 192.7)
- added C29: 0.1uF 25V, Capacitor_SMD:C_0603_1608Metric, F.Cu at (144.5, 193.5)
- added C3: 4.7uF, Capacitor_SMD:C_0603_1608Metric, F.Cu at (128.4, 195.2)
- added C30: 4.7uF, Capacitor_SMD:C_0603_1608Metric, F.Cu at (179.6, 162.5)
- added C31: 4.7uF, Capacitor_SMD:C_0603_1608Metric, F.Cu at (140.5, 195.7)
- added C32: 4.7uF 25V, Capacitor_SMD:C_0603_1608Metric, F.Cu at (144.5, 191.0)
- added C33: 4.7uF 25V, Capacitor_SMD:C_0603_1608Metric, F.Cu at (152.4, 186.0)
- added C34: 0.1uF, Capacitor_SMD:C_0603_1608Metric, F.Cu at (148.4, 188.5)
- added C35: 0.1uF, Capacitor_SMD:C_0603_1608Metric, F.Cu at (168.6, 173.5)
- added C4: 0.1uF, Capacitor_SMD:C_0603_1608Metric, F.Cu at (137.9, 190.6)
- added C5: 0.1uF, Capacitor_SMD:C_0603_1608Metric, F.Cu at (132.5, 193.1)
- added C6: 4.7uF, Capacitor_SMD:C_0603_1608Metric, F.Cu at (144.3, 186.0)
- added C7: 0.1uF, Capacitor_SMD:C_0603_1608Metric, F.Cu at (136.5, 193.1)
- added C8: 0.1uF, Capacitor_SMD:C_0603_1608Metric, F.Cu at (132.5, 195.7)
- added C9: 0.1uF, Capacitor_SMD:C_0603_1608Metric, F.Cu at (175.5, 162.5)
- added D1: MBR0520LT1G, Diode_SMD:D_SOD-123, F.Cu at (176.4, 159.6)
- added L1: 10uH CBC2518T100M, Inductor_SMD:L_1206_3216Metric_Pad1.42x1.75mm_HandSolder, F.Cu at (123.5, 194.6)
- added OLED1: UG-9664HDDAG01, myfootprint:UG-9664HDDAG01, B.Cu at (113.0, 146.0)
- added OLED2: UG-9664HDDAG01, myfootprint:UG-9664HDDAG01, B.Cu at (171.8, 146.0)
- added R1: 0, Resistor_SMD:R_0603_1608Metric, F.Cu at (165.2, 183.1)
- added R10: 0, Resistor_SMD:R_0603_1608Metric, F.Cu at (152.5, 193.5)
- added R11: 0, Resistor_SMD:R_0603_1608Metric, F.Cu at (172.6, 173.5)
- added R12: 4.7k, Resistor_SMD:R_0603_1608Metric, F.Cu at (152.5, 191.0)
- added R13: 4.7k, Resistor_SMD:R_0603_1608Metric, F.Cu at (179.6, 165.0)
- added R14: 4.7k, Resistor_SMD:R_0603_1608Metric, F.Cu at (161.2, 183.1)
- added R15: 4.7k, Resistor_SMD:R_0603_1608Metric, F.Cu at (148.5, 196.0)
- added R16: 0, Resistor_SMD:R_0603_1608Metric, F.Cu at (165.2, 180.5)
- added R17: 51k, Resistor_SMD:R_0603_1608Metric, F.Cu at (156.5, 196.0)
- added R18: 0, Resistor_SMD:R_0603_1608Metric, F.Cu at (169.2, 181.0)
- added R19: 4.7k, Resistor_SMD:R_0603_1608Metric, F.Cu at (165.2, 185.6)
- added R2: 0, Resistor_SMD:R_0603_1608Metric, F.Cu at (169.2, 178.5)
- added R20: 4.7k, Resistor_SMD:R_0603_1608Metric, F.Cu at (173.2, 176.0)
- added R21: 140k, Resistor_SMD:R_0603_1608Metric, F.Cu at (179.6, 170.0)
- added R22: 13.3k, Resistor_SMD:R_0603_1608Metric, F.Cu at (160.4, 188.1)
- added R23: 0, Resistor_SMD:R_0603_1608Metric, F.Cu at (156.5, 193.5)
- added R24: 1.1M, Resistor_SMD:R_0603_1608Metric, F.Cu at (176.6, 172.5)
- added R25: 1.1M, Resistor_SMD:R_0603_1608Metric, F.Cu at (156.4, 186.0)
- added R26: 0, Resistor_SMD:R_0603_1608Metric, F.Cu at (154.4, 116.2)
- added R3: 0, Resistor_SMD:R_0603_1608Metric, F.Cu at (152.5, 196.0)
- added R4: 0, Resistor_SMD:R_0603_1608Metric, F.Cu at (161.2, 185.6)
- added R5: 4.7k, Resistor_SMD:R_0603_1608Metric, F.Cu at (179.6, 167.5)
- added R6: 4.7k, Resistor_SMD:R_0603_1608Metric, F.Cu at (169.2, 176.0)
- added R7: 0, Resistor_SMD:R_0603_1608Metric, F.Cu at (173.2, 178.5)
- added R8: 0, Resistor_SMD:R_0603_1608Metric, F.Cu at (175.5, 170.0)
- added R9: 0, Resistor_SMD:R_0603_1608Metric, F.Cu at (156.4, 188.5)
- added TP1: TP_GND, TestPoint:TestPoint_Plated_Hole_D2.0mm, F.Cu at (140.0, 187.1)
- added TP2: TestPoint, TestPoint:TestPoint_Pad_D1.0mm, F.Cu at (160.1, 193.4)
- added U1: AP7361C-33E, Package_TO_SOT_SMD:SOT-223-3_TabPin2, F.Cu at (118.0, 188.8)
- added U2: SN74AVC4T245PW, Package_SO:TSSOP-16_4.4x5mm_P0.65mm, F.Cu at (127.4, 188.2)
- added U3: PCA9306DCTR, myfootprint:PCA9306DCTR, F.Cu at (129.4, 126.0)
- added U4: PCA9306DCTR, myfootprint:PCA9306DCTR, F.Cu at (155.6, 126.3)
- added U5: LM2733XMF, Package_TO_SOT_SMD:SOT-23-5_HandSoldering, F.Cu at (153.5, 138.9)
- added U6: BU90R104, Package_QFP:TQFP-64_10x10mm_P0.5mm, F.Cu at (134.3, 146.3)
- added U7: SS-MPU-9250, myfootprint:SS-MPU-9250, F.Cu at (142.5, 121.7)
Connections:
- J1 pad 1: (no net) -> /HS_SPI1_MOSI
- J1 pad 10: (no net) -> /HS_CSI0_D0_N
- J1 pad 11: (no net) -> /HS_SPI1_MISO
- J1 pad 12: (no net) -> GND
- J1 pad 13: (no net) -> GND
- J1 pad 14: (no net) -> /HS_CSI0_D1_P
- J1 pad 15: (no net) -> /HS_CSI0_MCLK
- J1 pad 16: (no net) -> /HS_CSI0_D1_N
- J1 pad 17: (no net) -> /HS_CSI1_MCLK
- J1 pad 18: (no net) -> GND
- J1 pad 19: (no net) -> GND
- J1 pad 2: (no net) -> /HS_CSI0_CLK_P
- J1 pad 20: (no net) -> /HS_CSI0_D2_P
- J1 pad 21: (no net) -> /HS_DSI_CLK_P
- J1 pad 22: (no net) -> /HS_CSI0_D2_N
- J1 pad 23: (no net) -> /HS_DSI_CLK_N
- J1 pad 24: (no net) -> GND
- J1 pad 25: (no net) -> GND
- J1 pad 26: (no net) -> /HS_CSI0_D3_P
- J1 pad 27: (no net) -> /HS_DSI_D0_P
- J1 pad 28: (no net) -> /HS_CSI0_D3_N
- J1 pad 29: (no net) -> /HS_DSI_D0_N
- J1 pad 3: (no net) -> Net-(J1-Pad3)
- J1 pad 30: (no net) -> GND
- J1 pad 31: (no net) -> GND
- J1 pad 32: (no net) -> /HS_I2C2_SCL
- J1 pad 33: (no net) -> /HS_DSI_D1_P
- J1 pad 34: (no net) -> /HS_I2C2_SDA
- J1 pad 35: (no net) -> /HS_DSI_D1_N
- J1 pad 36: (no net) -> /HS_I2C3_SCL
- J1 pad 37: (no net) -> GND
- J1 pad 38: (no net) -> /HS_I2C3_SDA
- J1 pad 39: (no net) -> /HS_DSI_D2_P
- J1 pad 4: (no net) -> /HS_CSI0_CLK_N
- J1 pad 40: (no net) -> GND
- J1 pad 41: (no net) -> /HS_DSI_D2_N
- J1 pad 42: (no net) -> /HS_CSI1_D0_P
- J1 pad 43: (no net) -> GND
- J1 pad 44: (no net) -> /HS_CSI1_D0_N
- J1 pad 45: (no net) -> /HS_DSI_D3_P
- J1 pad 46: (no net) -> GND
- J1 pad 47: (no net) -> /HS_DSI_D3_N
- J1 pad 48: (no net) -> /HS_CSI1_D1_P
- J1 pad 49: (no net) -> GND
- J1 pad 5: (no net) -> Net-(J1-Pad5)
- J1 pad 50: (no net) -> /HS_CSI1_D1_N
- J1 pad 51: (no net) -> /HS_USB2D3_P
- J1 pad 52: (no net) -> GND
- J1 pad 53: (no net) -> /HS_USB2D3_N
- J1 pad 54: (no net) -> /HS_CSI1_CLK_P
- J1 pad 55: (no net) -> GND
- J1 pad 56: (no net) -> /HS_CSI1_CLK_N
- J1 pad 57: (no net) -> Net-(J1-Pad57)
- J1 pad 58: (no net) -> GND
- J1 pad 59: (no net) -> Net-(J1-Pad59)
- J1 pad 6: (no net) -> GND
- J1 pad 60: (no net) -> Net-(J1-Pad60)
- J1 pad 7: (no net) -> /HS_SPI1_CS
- J1 pad 8: (no net) -> /HS_CSI0_D0_P
- J1 pad 9: (no net) -> /HS_SPI1_SCLK
- J2 pad 1: (no net) -> GND
- J2 pad 10: (no net) -> /LS_SPI0_MISO
- J2 pad 11: (no net) -> /LS_GPIO_4
- J2 pad 12: (no net) -> /LS_SPI0_CS
- J2 pad 13: (no net) -> /LS_GPIO_5
- J2 pad 14: (no net) -> /LS_SPI0_MOSI
- J2 pad 15: (no net) -> /LS_I2C0_SCL
- J2 pad 16: (no net) -> /LS_GPIO_9
- J2 pad 17: (no net) -> /LS_I2C0_SDA
- J2 pad 18: (no net) -> /LS_GPIO_10
- J2 pad 19: (no net) -> /LS_I2C1_SCL
- J2 pad 2: (no net) -> GND
- J2 pad 20: (no net) -> /LS_GPIO_11
- J2 pad 21: (no net) -> /LS_I2C1_SDA
- J2 pad 22: (no net) -> /LS_GPIO_12
- J2 pad 23: (no net) -> /LS_PS_GPIO_0
- J2 pad 24: (no net) -> /LS_PS_GPIO_1
- J2 pad 25: (no net) -> /LS_PS_GPIO_2
- J2 pad 26: (no net) -> /LS_PS_GPIO_3
- J2 pad 27: (no net) -> /LS_PS_GPIO_4
- J2 pad 28: (no net) -> /LS_PS_GPIO_5
- J2 pad 29: (no net) -> /LS_GPIO_6
- J2 pad 3: (no net) -> /LS_GPIO_0
- J2 pad 30: (no net) -> /LS_GPIO_13
- J2 pad 31: (no net) -> /LS_GPIO_7
- J2 pad 32: (no net) -> /LS_GPIO_14
- J2 pad 33: (no net) -> /LS_GPIO_8
- J2 pad 34: (no net) -> /LS_GPIO_15
- J2 pad 35: (no net) -> +1V8
- J2 pad 36: (no net) -> /VSYS_IN0
- J2 pad 37: (no net) -> +5V
- J2 pad 38: (no net) -> /VSYS_IN1
- J2 pad 39: (no net) -> GND
- J2 pad 4: (no net) -> /PWR_PB_N
- J2 pad 40: (no net) -> GND
- J2 pad 5: (no net) -> /LS_GPIO_1
- J2 pad 6: (no net) -> /RST_PB_N
- J2 pad 7: (no net) -> /LS_GPIO_2
- J2 pad 8: (no net) -> /LS_SPI0_SCLK
- J2 pad 9: (no net) -> /LS_GPIO_3
- J3 pad 1: (no net) -> GND
- J3 pad 10: (no net) -> GND
- J3 pad 11: (no net) -> /CAM0_GPIO
- J3 pad 12: (no net) -> /CAM0_CLK
- J3 pad 13: (no net) -> /CAM0_SCL
- J3 pad 14: (no net) -> /CAM0_SDA
- J3 pad 15: (no net) -> +3V3
- J3 pad 2: (no net) -> /HS_CSI0_D0_N
- J3 pad 3: (no net) -> /HS_CSI0_D0_P
- J3 pad 4: (no net) -> GND
- J3 pad 5: (no net) -> /HS_CSI0_D1_N
- J3 pad 6: (no net) -> /HS_CSI0_D1_P
- J3 pad 7: (no net) -> GND
- J3 pad 8: (no net) -> /HS_CSI0_CLK_N
- J3 pad 9: (no net) -> /HS_CSI0_CLK_P
- J4 pad 1: (no net) -> GND
- J4 pad 10: (no net) -> GND
- J4 pad 11: (no net) -> /CAM1_GPIO
- J4 pad 12: (no net) -> /CAM1_CLK
- J4 pad 13: (no net) -> /CAM1_SCL
- J4 pad 14: (no net) -> /CAM1_SDA
- J4 pad 15: (no net) -> +3V3
- J4 pad 2: (no net) -> /HS_CSI1_D0_N
- J4 pad 3: (no net) -> /HS_CSI1_D0_P
- J4 pad 4: (no net) -> GND
- J4 pad 5: (no net) -> /HS_CSI1_D1_N
- J4 pad 6: (no net) -> /HS_CSI1_D1_P
- J4 pad 7: (no net) -> GND
- J4 pad 8: (no net) -> /HS_CSI1_CLK_N
- J4 pad 9: (no net) -> /HS_CSI1_CLK_P
Routing:
- net /HS_CSI1_D0_P: track 0.00 -> 42.4 mm, vias 0 -> 1
- net /HS_CSI1_D0_N: track 0.00 -> 42.4 mm, vias 0 -> 1
- net /HS_CSI1_CLK_P: track 0.00 -> 42.1 mm, vias 0 -> 1
- net /OLED1_D7: track 0.00 -> 42.0 mm, vias 0 -> 1
- net /HS_CSI1_CLK_N: track 0.00 -> 42.0 mm, vias 0 -> 1
- net /HS_CSI1_D1_P: track 0.00 -> 41.9 mm, vias 0 -> 1
- net /HS_CSI1_D1_N: track 0.00 -> 41.9 mm, vias 0 -> 1
- net /OLED1_D6: track 0.00 -> 41.6 mm, vias 0 -> 1
- net /OLED1_D5: track 0.00 -> 41.5 mm, vias 0 -> 1
- net /OLED1_D4: track 0.00 -> 39.7 mm, vias 0 -> 1
- net /OLED1_D3: track 0.00 -> 39.1 mm, vias 0 -> 1
- net /OLED1_D0: track 0.00 -> 38.6 mm, vias 0 -> 1
- net /OLED1_D2: track 0.00 -> 38.2 mm, vias 0 -> 1
- net /OLED1_D1: track 0.00 -> 37.4 mm, vias 0 -> 1
- net /HS_I2C3_SCL: track 0.00 -> 31.5 mm, vias 0 -> 1
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
Commit message: update
Parts:
- moved L1 61.3 mm to (151.2, 140.0), turned to 90 degrees
- moved R17 59.9 mm to (154.3, 136.2)
- moved R22 48.7 mm to (157.2, 139.5), turned to 90 degrees
- moved R23 47.1 mm to (157.2, 146.4), turned to 270 degrees
- moved C14 46.2 mm to (154.3, 144.9), turned to 180 degrees
- moved R16 42.3 mm to (159.0, 138.7), turned to 270 degrees
- moved C13 40.4 mm to (154.3, 138.2)
- moved C15 39.8 mm to (154.3, 146.6), turned to 180 degrees
- moved R21 35.2 mm to (157.2, 142.8), turned to 90 degrees
- moved D1 29.2 mm to (151.2, 145.0), turned to 90 degrees
- moved U5 2.68 mm to (154.4, 141.4), turned to 90 degrees
Connections:
- U6 pad 20: Net-(TP2-Pad1) -> /PWR_EN
Routing:
- net VCC: track 0.00 -> 82.2 mm, vias 0 -> 2
- net /OLED1_D0: track 38.6 -> 17.3 mm, vias 1 -> 0
- net /OLED1_D1: track 37.4 -> 22.7 mm, vias 1 -> 0
- net GND: track 0.07 -> 11.5 mm
- net /VCC_OUT: track 0.00 -> 9.87 mm
- net /VCC_SHDN: track 0.00 -> 9.35 mm
- net /VCC_SW: track 0.00 -> 7.69 mm
- net +5V: track 0.00 -> 7.25 mm
- net /VCC_FB: track 0.00 -> 6.17 mm
- net /OLED1_D3: track 39.1 -> 33.1 mm
- net /OLED1_D2: track 38.2 -> 32.5 mm
- net /HS_I2C2_SCL: track 18.4 -> 13.8 mm
- net /CAM0_SCL: track 19.9 -> 16.7 mm
- net /CAM0_SDA: track 15.6 -> 18.4 mm
- net +1V8: track 0.00 -> 1.82 mm, vias 0 -> 1
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
Commit message: update
Parts:
- added C3: 10uF, Capacitor_SMD:C_0603_1608Metric, F.Cu at (144.2, 110.7)
- added C6: 22uF, Capacitor_SMD:C_0603_1608Metric, F.Cu at (138.6, 114.3)
- added L2: 2.2uH MLZ2012A2R2MT, Inductor_SMD:L_0805_2012Metric, F.Cu at (135.2, 113.2)
- added R27: 100k, Resistor_SMD:R_0603_1608Metric, F.Cu at (133.0, 110.7)
- added R28: 562k, Resistor_SMD:R_0603_1608Metric, F.Cu at (137.1, 108.6)
- added R29: 180k, Resistor_SMD:R_0603_1608Metric, F.Cu at (140.6, 108.6)
- added R30: 0, Resistor_SMD:R_0603_1608Metric, F.Cu at (132.2, 114.2)
- added SW1: SW_Push, Button_Switch_SMD:SW_Push_1P1T_NO_CK_KMR2, F.Cu at (180.7, 109.4)
- added SW2: SW_Push, Button_Switch_SMD:SW_Push_1P1T_NO_CK_KMR2, F.Cu at (173.0, 109.4)
- added U1: TPS62160DGK, Package_SO:MSOP-8_3x3mm_P0.65mm, F.Cu at (140.1, 111.5)
- C16, C18, C19, C20, C21: moved to B.Cu
- moved U1 88.1 mm to (156.2, 109.5)
- moved TP1 82.5 mm to (103.2, 113.2)
- moved U2 77.4 mm to (122.7, 110.9)
- moved R15 75.5 mm to (156.3, 120.9), turned to 90 degrees
- moved R12 75.1 mm to (126.5, 120.5), turned to 270 degrees
- moved C8 68.9 mm to (127.7, 126.9)
- moved R19 68.3 mm to (159.7, 117.5)
- moved R13 67.9 mm to (128.2, 120.5), turned to 270 degrees
- moved R6 67.7 mm to (130.5, 120.5), turned to 90 degrees
- moved R5 66.7 mm to (132.2, 120.5), turned to 90 degrees
- moved C10 66.2 mm to (157.4, 123.6), turned to 180 degrees
- moved R14 62.5 mm to (154.7, 120.9), turned to 90 degrees
- moved R20 61.8 mm to (159.7, 115.7)
- moved R18 61.1 mm to (158.0, 120.9), turned to 270 degrees
- moved C17 58.6 mm to (133.4, 138.6), turned to 180 degrees
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Connections:
- U2 pad 6: /HS_CSI0_MCLK -> /LS_GPIO_2
- U2 pad 7: /HS_CSI1_MCLK -> /LS_GPIO_3
Routing:
- net /CAM1_SCL: track 0.00 -> 47.4 mm
- net /CAM1_SDA: track 0.00 -> 47.3 mm, vias 0 -> 2
- net +1V8: track 1.82 -> 48.5 mm, vias 1 -> 3
- net GND: track 11.5 -> 40.8 mm, vias 0 -> 4
- net /OLED1_D0: track 17.3 -> 40.2 mm, vias 0 -> 1
- net Net-(C6-Pad1): track 0.00 -> 16.5 mm, vias 0 -> 2
- net /OLED1_D1: track 22.7 -> 38.9 mm, vias 0 -> 1
- net +3V3: track 27.3 -> 41.6 mm, vias 1 -> 4
- net +5V: track 7.25 -> 16.9 mm
- net /OLED1_D3: track 33.1 -> 40.8 mm
- net /OLED1_D2: track 32.5 -> 39.9 mm
- net /HS_I2C3_SDA: track 29.6 -> 36.7 mm
- net Net-(R27-Pad1): track 0.00 -> 6.77 mm, vias 0 -> 2
- net /HS_I2C3_SCL: track 29.7 -> 35.8 mm
- net /CAM0_SDA: track 18.4 -> 13.6 mm
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
Commit message: update
Parts:
- removed the C3 at (128.4, 195.2)
- removed the C6 at (144.3, 186.0)
- removed TP2: TestPoint, TestPoint:TestPoint_Pad_D1.0mm
- removed the U1 at (140.1, 111.5)
- removed the U1 at (156.2, 109.5)
- added D1: SML-512MWT86, LED_SMD:LED_0603_1608Metric_Pad1.05x0.95mm_HandSolder, F.Cu at (166.0, 111.5)
- added D2: SML-512MWT86, LED_SMD:LED_0603_1608Metric_Pad1.05x0.95mm_HandSolder, F.Cu at (168.0, 111.5)
- added D3: SML-512MWT86, LED_SMD:LED_0603_1608Metric_Pad1.05x0.95mm_HandSolder, F.Cu at (170.0, 111.5)
- added D4: SML-512MWT86, LED_SMD:LED_0603_1608Metric_Pad1.05x0.95mm_HandSolder, F.Cu at (172.0, 111.5)
- added R31: 4.7k, Resistor_SMD:R_0603_1608Metric, F.Cu at (153.0, 111.6)
- added R32: 4.7k, Resistor_SMD:R_0603_1608Metric, F.Cu at (154.8, 111.6)
- added R33: 4.7k, Resistor_SMD:R_0603_1608Metric, F.Cu at (156.6, 111.7)
- added R34: 4.7k, Resistor_SMD:R_0603_1608Metric, F.Cu at (158.2, 111.7)
- added R35: 4.7k, Resistor_SMD:R_0603_1608Metric, F.Cu at (164.7, 106.2)
- added R36: 4.7k, Resistor_SMD:R_0603_1608Metric, F.Cu at (174.9, 106.2)
- added R37: 0, Resistor_SMD:R_0603_1608Metric, F.Cu at (115.3, 117.7)
- added R38: 0, Resistor_SMD:R_0603_1608Metric, F.Cu at (174.0, 128.6)
- added R39: <0>, Resistor_SMD:R_0603_1608Metric, F.Cu at (118.0, 117.7)
- added R40: <0>, Resistor_SMD:R_0603_1608Metric, F.Cu at (120.1, 117.7)
- added R41: <0>, Resistor_SMD:R_0603_1608Metric, F.Cu at (175.9, 128.6)
- added R42: <0>, Resistor_SMD:R_0603_1608Metric, F.Cu at (177.6, 128.6)
- added SW3: KMR213G LFG, Button_Switch_SMD:SW_Push_1P1T_NO_CK_KMR2, F.Cu at (107.7, 112.4)
- added SW4: KMR213G LFG, Button_Switch_SMD:SW_Push_1P1T_NO_CK_KMR2, F.Cu at (113.0, 112.4)
- added SW5: GDH04S04, Button_Switch_SMD:SW_DIP_SPSTx04_Slide_Omron_A6H-4101_W6.15mm_P1.27mm, F.Cu at (155.8, 105.3)
- added U1: TPS62160DGK, myfootprint:TPS62160DGK, F.Cu at (140.2, 111.5)
- C11, C12, C22, C23, C24, C25, C26, C27, C28, C29, C30, C31, C32, C33, C34, C35, R24, R25: moved to B.Cu
- R10, R7, R8, R9: value 0 -> 10
- SW1, SW2: value SW_Push -> KMR213G LFG
- moved R3 92.3 mm to (117.1, 110.8), turned to 180 degrees
- moved R4 85.4 mm to (117.1, 112.5), turned to 180 degrees
- moved C7 84.9 mm to (124.8, 109.0), turned to 180 degrees
- moved C4 83.5 mm to (120.3, 109.0)
- moved C1 83.5 mm to (148.2, 107.5)
- moved C2 82.4 mm to (148.2, 109.5)
- moved R1 81.2 mm to (129.1, 110.3)
- moved R10 80.9 mm to (172.0, 115.0), turned to 90 degrees
- moved R2 77.6 mm to (129.1, 112.0)
- moved TP1 75.9 mm to (179.1, 113.2)
- moved R9 74.7 mm to (170.0, 115.0), turned to 90 degrees
- moved C11 74.7 mm to (117.5, 122.1), turned to 180 degrees
- moved C30 74.6 mm to (108.6, 139.5)
- moved R24 73.5 mm to (111.2, 139.1), turned to 270 degrees
- moved C12 69.8 mm to (176.5, 122.1), turned to 180 degrees
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- renumbered D1 to D5
Connections:
- C30 pad 1: Net-(C30-Pad1) -> +3V3
- C31 pad 1: Net-(C31-Pad1) -> +3V3
- C34 pad 1: Net-(C30-Pad1) -> +3V3
- C35 pad 1: Net-(C31-Pad1) -> +3V3
- OLED1 pad 4: Net-(C30-Pad1) -> +3V3
- OLED2 pad 4: Net-(C31-Pad1) -> +3V3
- R10 pad 1: /CAM1_CLK -> GND
- R10 pad 2: Net-(R10-Pad2) -> Net-(D4-Pad1)
- R7 pad 1: /CAM0_GPIO -> GND
- R7 pad 2: Net-(R7-Pad2) -> Net-(D1-Pad1)
- R8 pad 1: /CAM1_GPIO -> GND
- R8 pad 2: Net-(R8-Pad2) -> Net-(D2-Pad1)
- R9 pad 1: /CAM0_CLK -> GND
- R9 pad 2: Net-(R9-Pad2) -> Net-(D3-Pad1)
- SW1 pad 1: /PWR_PB_N -> /LS_GPIO_8
- SW1 pad 2: GND -> +1V8
- SW2 pad 1: /RST_PB_N -> /LS_GPIO_9
- SW2 pad 2: GND -> +1V8
- U2 pad 10: Net-(R10-Pad2) -> /LS_3V3_GPIO_1
- U2 pad 11: Net-(R9-Pad2) -> /LS_3V3_GPIO_0
- U2 pad 12: Net-(R8-Pad2) -> /LS_3V3_PS_GPIO_1
- U2 pad 13: Net-(R7-Pad2) -> /LS_3V3_PS_GPIO_0
- U2 pad 4: /LS_GPIO_0 -> /LS_PS_GPIO_0
- U2 pad 5: /LS_GPIO_1 -> /LS_PS_GPIO_1
- U2 pad 6: /LS_GPIO_2 -> /LS_GPIO_0
- U2 pad 7: /LS_GPIO_3 -> /LS_GPIO_1
Routing:
- net GND: track 40.8 -> 750.5 mm, vias 4 -> 55
- net +3V3: track 41.6 -> 370.5 mm, vias 4 -> 19
- net +1V8: track 48.5 -> 155.5 mm, vias 3 -> 5
- net +5V: track 16.9 -> 119.6 mm, vias 0 -> 1
- net /OLED_DC: track 0.00 -> 85.0 mm, vias 0 -> 2
- net /OLED_RW: track 0.00 -> 80.4 mm, vias 0 -> 4
- net /LS_3V3_PS_GPIO_1: track 0.00 -> 79.8 mm, vias 0 -> 2
- net /LS_3V3_GPIO_1: track 0.00 -> 77.8 mm, vias 0 -> 2
- net /OLED_E: track 0.00 -> 75.7 mm, vias 0 -> 4
- net /LS_3V3_PS_GPIO_0: track 0.00 -> 64.7 mm, vias 0 -> 2
- net /LS_GPIO_9: track 0.00 -> 58.9 mm, vias 0 -> 1
- net /LS_3V3_GPIO_0: track 0.00 -> 56.4 mm, vias 0 -> 2
- net /LS_GPIO_4: track 0.00 -> 44.1 mm, vias 0 -> 2
- net /OLED1_BS2: track 0.00 -> 40.1 mm, vias 0 -> 3
- net /LS_GPIO_5: track 0.00 -> 40.0 mm, vias 0 -> 2
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Other:
- board text added: "PWR"
- board text added: "RST"

Commit message: update
Parts:
- TP1: footprint TestPoint:TestPoint_Plated_Hole_D2.0mm -> TestPoint:TestPoint_Loop_D1.80mm_Drill1.0mm_Beaded
- moved C32 2.11 mm to (116.0, 142.0)
- moved TP1 0.22 mm to (179.2, 113.0)
Routing:
- net GND: track 750.5 -> 811.5 mm, vias 55 -> 155
- net +1V8: track 155.5 -> 184.3 mm, vias 5 -> 6
- net /LS_3V3_PS_GPIO_0: track 64.7 -> 54.2 mm
- net /OLED_E: track 75.7 -> 78.9 mm
- net /OLED0_VCOMH: track 4.17 -> 6.28 mm
- net /OLED0_D6: track 14.9 -> 16.5 mm
- net /OLED1_D7: track 46.4 -> 44.9 mm
- net /OLED1_D6: track 45.6 -> 44.2 mm
- net +3V3: track 370.5 -> 371.4 mm, vias 19 -> 20
- net /OLED0_RES: track 22.0 -> 22.8 mm
- net (no net): vias 0 -> 1
- added copper zone on B.Cu, net GND
- added copper zone on F.Cu, net GND
Other:
- board text added: "GND"

Commit message: update
Parts:
- added C36: 0.1uF, Capacitor_SMD:C_0603_1608Metric, F.Cu at (130.9, 129.5)
- added TP2: TP_GND, TestPoint:TestPoint_Pad_D1.0mm, F.Cu at (148.6, 149.6)
- added X1: SIT2024BA-S3-18E-25.000000G, Package_TO_SOT_SMD:SOT-23-5_HandSoldering, F.Cu at (131.7, 132.1)
- C6: value 22uF -> 10uF
- L2: value 2.2uH MLZ2012A2R2MT -> 2.2uH_2012
- R10, R7, R8, R9: value 10 -> 100
- R27: value 100k -> 0
- R28: value 562k -> 0
- R29: value 180k -> 0
- U1: value TPS62160DGK -> LM3671MF-3.3; footprint myfootprint:TPS62160DGK -> Package_TO_SOT_SMD:TSOT-23-5
- moved R27 43.3 mm to (145.0, 152.3), turned to 0 degrees
- moved R28 42.8 mm to (145.0, 150.7), turned to 0 degrees
- moved R29 40.7 mm to (145.0, 149.1), turned to 0 degrees
- moved C3 1.20 mm to (143.3, 111.5)
- moved U1 0.19 mm to (140.0, 111.4)
Connections:
- R27 pad 2: Net-(C6-Pad1) -> +3V3
- R28 pad 2: Net-(C6-Pad1) -> +3V3
- R29 pad 1: GND -> Net-(R29-Pad1)
- R29 pad 2: Net-(R28-Pad1) -> +3V3
- U1 pad 1: GND -> +5V
- U1 pad 2: +5V -> GND
- U1 pad 4: GND -> Net-(C6-Pad1)
- U1 pad 5: Net-(R28-Pad1) -> Net-(L2-Pad2)
- U6 pad 3: +3V3 -> Net-(R27-Pad1)
- U6 pad 4: +3V3 -> Net-(R28-Pad1)
- U6 pad 5: +3V3 -> Net-(R29-Pad1)
Routing:
- net +1V8: track 184.3 -> 195.8 mm, vias 6 -> 8
- net /HS_CSI0_MCLK: track 0.00 -> 9.09 mm, vias 0 -> 1
- net GND: track 811.5 -> 820.3 mm, vias 155 -> 160
- net Net-(R29-Pad1): track 0.00 -> 5.16 mm
- net +3V3: track 371.4 -> 376.1 mm
- net +5V: track 119.6 -> 124.1 mm
- net Net-(C6-Pad1): track 16.4 -> 12.9 mm, vias 2 -> 0
- net /OLED_DC: track 84.6 -> 88.1 mm
- net /OLED_RW: track 80.6 -> 83.1 mm
- net Net-(R28-Pad1): track 3.89 -> 5.81 mm
- net Net-(L2-Pad2): track 2.97 -> 3.52 mm
- net Net-(R27-Pad1): track 6.77 -> 6.24 mm, vias 2 -> 0
