File: ultra96v2_glasses.kicad_pcb (KiCad board)
At the start: 2 copper layers, 85 x 54 mm, 110 parts, among them J1 61083-063402LF, J2 10075024-G01-20ULF, J3 1-1734248-5, J4 1-1734248-5, SW1 KMR213G LFG, SW2 KMR213G LFG, SW3 KMR213G LFG, SW4 KMR213G LFG, SW5 GDH04S04, U1 LM3671MF-3.3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

Commit message: update
Parts:
- J1: value 61083-063402LF -> 61083-064402LF
- J3, J4: footprint myfootprint:55510-140LF -> myfootprint:55510-140LF_handsolder
- moved R40 1.80 mm to (121.9, 117.6)
- moved R37 0.90 mm to (115.3, 116.8)
- moved R39 0.80 mm to (118.0, 116.9)
Routing:
- net GND: track 820.3 -> 708.9 mm, vias 160 -> 140
- net /CAM0_SDA: track 13.6 -> 8.23 mm
- net /CAM0_SCL: track 15.0 -> 10.1 mm
- net /HS_CSI0_D1_P: track 29.4 -> 26.2 mm
- net /HS_CSI0_D0_P: track 29.6 -> 26.4 mm
- net /HS_CSI0_CLK_N: track 29.5 -> 26.3 mm
- net /HS_CSI0_D0_N: track 29.6 -> 26.9 mm
- net /HS_CSI0_CLK_P: track 29.5 -> 26.8 mm
- net /HS_CSI0_D1_N: track 29.4 -> 27.2 mm
- net /CAM0_GPIO: track 12.2 -> 10.5 mm
- net /CAM0_CLK: track 13.3 -> 14.1 mm

Commit message: update
Parts:
- removed OLED2: UG-9664HDDAG01, myfootprint:UG-9664HDDAG01
- moved R14 2.61 mm to (154.9, 118.3)
- moved R26 2.61 mm to (152.8, 118.3)
- moved R15 2.61 mm to (156.5, 118.3)
- moved R18 2.61 mm to (158.2, 118.3)
- moved C9 2.61 mm to (153.4, 120.9)
- moved C10 2.61 mm to (157.6, 121.0)
- moved U4 2.61 mm to (155.8, 123.7)
- moved C11 1.95 mm to (117.8, 120.2)
- moved R19 1.60 mm to (159.7, 115.9)
- moved R38 1.55 mm to (175.6, 128.6)
- moved R20 1.43 mm to (159.7, 114.3)
- moved R42 1.40 mm to (179.0, 128.6)
- moved R41 1.38 mm to (177.3, 128.6)
- moved R39 0.93 mm to (117.0, 116.8)
- moved R40 0.55 mm to (122.1, 117.1), turned to 0 degrees
Routing:
- net GND: track 708.9 -> 752.8 mm, vias 140 -> 139
- net /CAM0_SDA: track 8.23 -> 19.0 mm
- net /CAM0_SCL: track 10.1 -> 20.4 mm, vias 0 -> 2
- net /HS_CSI0_D1_P: track 26.2 -> 32.3 mm
- net /HS_CSI0_CLK_N: track 26.3 -> 32.2 mm
- net /HS_CSI0_D0_N: track 26.9 -> 32.3 mm
- net /HS_CSI0_CLK_P: track 26.8 -> 32.2 mm
- net /HS_CSI0_D1_N: track 27.2 -> 32.5 mm
- net /HS_CSI0_D0_P: track 26.4 -> 31.6 mm
- net /CAM1_CLK: track 5.36 -> 9.95 mm
- net /CAM0_CLK: track 14.1 -> 18.3 mm, vias 2 -> 1
- net /CAM1_GPIO: track 6.91 -> 11.1 mm
- net +3V3: track 376.1 -> 372.2 mm, vias 20 -> 21
- net +1V8: track 195.8 -> 192.5 mm
- net Net-(R26-Pad1): track 4.16 -> 7.34 mm, vias 0 -> 1
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Other:
- board text removed: "ULTRA96-GLASSES Rev.1 (C) Ryuji Fuchikami"

Commit message: rev2
Parts:
- added OLED2: UG-9664HDDAG01, myfootprint:UG-9664HDDAG01, B.Cu at (171.8, 146.0)
Other:
- board text added: "96-GLASSES Rev.2 (C) Ryuji Fuchikami"

Commit message: update rev3
Parts:
- added R43: 100, Resistor_SMD:R_0603_1608Metric, F.Cu at (134.3, 140.9)
- added R44: 100, Resistor_SMD:R_0603_1608Metric, F.Cu at (136.7, 139.4)
- added R45: 100, Resistor_SMD:R_0603_1608Metric, F.Cu at (139.2, 140.9)
- C17, R27: moved to B.Cu
- R28, R29: value 0 -> 100
- U6: value BU90R104 -> THC63LVDR84C; footprint Package_QFP:TQFP-64_10x10mm_P0.5mm -> Package_SO:TSSOP-56_6.1x14mm_P0.5mm
- moved TP2 47.3 mm to (101.3, 151.3)
- moved R27 19.1 mm to (127.8, 144.0), turned to 180 degrees
- moved R28 18.4 mm to (129.4, 140.9), turned to 180 degrees
- moved R29 16.3 mm to (131.9, 139.4), turned to 180 degrees
- moved C17 13.9 mm to (137.0, 151.5), turned to 0 degrees
- moved C19 12.7 mm to (140.3, 151.5), turned to 180 degrees
- moved C16 11.3 mm to (129.7, 151.5), turned to 0 degrees
- moved C21 9.43 mm to (130.6, 145.5), turned to 0 degrees
- moved C18 8.42 mm to (133.7, 151.5), turned to 0 degrees
- moved C20 6.25 mm to (134.6, 145.5), turned to 180 degrees
- moved U6 1.91 mm to (134.1, 147.8), turned to 270 degrees
- moved C28 1.62 mm to (123.2, 142.9)
Connections:
- R28 pad 1: Net-(R28-Pad1) -> /HS_DSI_CLK_N
- R28 pad 2: +3V3 -> /HS_DSI_CLK_P
- R29 pad 1: Net-(R29-Pad1) -> /HS_DSI_D0_N
- R29 pad 2: +3V3 -> /HS_DSI_D0_P
- U6 pad 1: GND -> /OLED1_BS1
- U6 pad 10: /OLED1_D4 -> /HS_DSI_D3_P
- U6 pad 11: /OLED1_D3 -> /HS_DSI_D2_N
- U6 pad 12: /OLED1_D2 -> /HS_DSI_D2_P
- U6 pad 13: /OLED1_D1 -> +3V3
- U6 pad 14: /OLED1_D0 -> GND
- U6 pad 15: /OLED1_RES -> /HS_DSI_D1_N
- U6 pad 16: GND -> /HS_DSI_D1_P
- U6 pad 17: /OLED1_CS -> /HS_DSI_D0_N
- U6 pad 18: /OLED1_BS2 -> /HS_DSI_D0_P
- U6 pad 19: /OLED1_BS1 -> /HS_DSI_CLK_N
- U6 pad 2: Net-(U6-Pad2) -> /OLED1_BS2
- U6 pad 20: /PWR_EN -> /HS_DSI_CLK_P
- U6 pad 21: /OLED_E -> GND
- U6 pad 22: Net-(U6-Pad22) -> GND
- U6 pad 24: Net-(U6-Pad24) -> GND
- U6 pad 25: Net-(U6-Pad25) -> Net-(R27-Pad1)
- U6 pad 27: Net-(U6-Pad27) -> /OLED0_D7
- U6 pad 28: Net-(U6-Pad28) -> GND
- U6 pad 29: Net-(U6-Pad29) -> /OLED0_RES
- U6 pad 3: Net-(R27-Pad1) -> /OLED_DC
- U6 pad 30: GND -> /OLED0_CS
- U6 pad 31: Net-(U6-Pad31) -> +3V3
- U6 pad 32: /OLED_RW -> /OLED0_BS2
- U6 pad 33: /OLED_DC -> /OLED0_BS1
- U6 pad 34: /OLED0_RES -> /OLED0_D0
- U6 pad 35: /OLED0_CS -> /OLED0_D1
- U6 pad 36: /OLED0_BS2 -> GND
- U6 pad 37: +3V3 -> /OLED0_D2
- U6 pad 38: /OLED0_BS1 -> /OLED0_D3
- U6 pad 39: /OLED0_D7 -> /OLED0_D4
- U6 pad 4: Net-(R28-Pad1) -> GND
- U6 pad 40: /OLED0_D6 -> +3V3
- U6 pad 42: /OLED0_D4 -> /OLED0_D6
- U6 pad 43: /OLED0_D3 -> /OLED1_D7
- U6 pad 45: /OLED0_D2 -> /OLED1_CS
- U6 pad 46: /OLED0_D1 -> /OLED1_RES
- U6 pad 47: /OLED0_D0 -> /OLED1_D0
- U6 pad 49: /HS_DSI_D0_N -> /OLED1_D1
- U6 pad 5: Net-(R29-Pad1) -> /OLED_RW
- U6 pad 50: /HS_DSI_D0_P -> /OLED1_D2
- U6 pad 51: /HS_DSI_D1_N -> /OLED1_D3
- U6 pad 52: /HS_DSI_D1_P -> GND
- U6 pad 53: +3V3 -> /OLED1_D6
- U6 pad 54: Net-(U6-Pad54) -> /OLED1_D5
- U6 pad 55: Net-(U6-Pad55) -> /OLED1_D4
- U6 pad 56: /HS_DSI_CLK_N -> +3V3
- U6 pad 6: /OLED1_D7 -> /OLED_E
- U6 pad 7: /OLED1_D6 -> /PWR_EN
- U6 pad 8: /OLED1_D5 -> GND
- U6 pad 9: +3V3 -> /HS_DSI_D3_N
Routing:
- net GND: track 752.8 -> 646.4 mm, vias 139 -> 118
- net /OLED_DC: track 88.1 -> 70.4 mm
- net +3V3: track 372.2 -> 357.3 mm, vias 21 -> 24
- net /OLED_RW: track 83.1 -> 70.4 mm, vias 4 -> 2
- net /HS_DSI_CLK_N: track 17.4 -> 7.33 mm
- net /OLED1_D7: track 44.9 -> 54.3 mm, vias 1 -> 4
- net /HS_DSI_CLK_P: track 17.2 -> 8.14 mm
- net /OLED_E: track 78.9 -> 71.1 mm, vias 4 -> 2
- net /HS_DSI_D1_P: track 14.2 -> 6.59 mm
- net /HS_DSI_D1_N: track 14.0 -> 6.96 mm
- net /OLED1_RES: track 35.0 -> 41.1 mm
- net /HS_DSI_D3_P: track 13.4 -> 7.59 mm
- net Net-(R28-Pad1): track 5.81 -> 0.00 mm
- net /HS_DSI_D0_N: track 13.3 -> 7.91 mm
- net Net-(R29-Pad1): track 5.16 -> 0.00 mm
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Other:
- board text added: "96-GLASSES Rev.3 (C) Ryuji Fuchikami"
- board text removed: "96-GLASSES Rev.2 (C) Ryuji Fuchikami"
